Commit message: test code for fish dynamically falls added

File: models/bowl/bowl.urdf (robot description, URDF)
Before this commit: robot bowl, 1 links, 0 joints
Links:
- link bowl: geometry collision mesh filename=package://bowl/bowl4.stl scale=.1 .1 .1; visual mesh filename=package://bowl/bowl4.dae scale=.1 .1 .1
