Commit message: RRT-bisec debugged and bowl added

File: models/triple_hook/triple_hook.urdf (robot description, URDF)
Before this commit: robot hook, 1 links, 0 joints
Links:
- link hook: geometry collision mesh filename=package://triple_hook/triple_hook.stl scale=0.05 0.05 0.05; visual mesh filename=package://triple_hook/triple_hook.dae scale=0.05 0.05 0.05

Commit message: fish with ring added

File: models/triple_hook/triple_hook.urdf (robot description, URDF)
Before this commit: robot hook, 1 links, 0 joints
Links:
- link hook: geometry collision mesh filename=package://triple_hook/triple_hook.stl scale=0.2 0.2 0.2; visual mesh filename=package://triple_hook/triple_hook.dae scale=0.2 0.2 0.2
