Commit message: fish with ringg added but BIT collision check not work with such thin things

File: models/fish/fishWithRing.xacro (robot description, xacro)
@@ -357,10 +357,10 @@
     <visual>
       <geometry>
-        <mesh filename="package://fish/ring.dae" scale=".02 .02 .02"/>
-      </geometry>
-    </visual>
-    <collision>
-      <geometry>
-        <mesh filename="package://fish/ring.stl" scale=".02 .02 .02"/>
+        <mesh filename="package://fish/ring2_vhacd.dae" scale=".02 .02 .02"/>
+      </geometry>
+    </visual>
+    <collision>
+      <geometry>
+        <mesh filename="package://fish/ring2_vhacd.OBJ" scale=".02 .02 .02"/>
       </geometry>
     </collision>

Commit message: fish clapaps ring works; starfish added

File: models/fish/fishWithRing.xacro (robot description, xacro)
@@ -357,10 +357,10 @@
     <visual>
       <geometry>
-        <mesh filename="package://fish/ring2_vhacd.dae" scale=".02 .02 .02"/>
-      </geometry>
-    </visual>
-    <collision>
-      <geometry>
-        <mesh filename="package://fish/ring2_vhacd.OBJ" scale=".02 .02 .02"/>
+        <mesh filename="package://fish/ring2_vhacd.dae" scale=".04 .04 .04"/>
+      </geometry>
+    </visual>
+    <collision>
+      <geometry>
+        <mesh filename="package://fish/ring2_vhacd.OBJ" scale=".04 .04 .04"/>
       </geometry>
     </collision>
