Commit message: gripper clenches starfish works

File: models/robotiq_3f_gripper_visualization/cfg/robotiq-3f-gripper_articulated.urdf (robot description, URDF)
Before this commit: robot robotiq-3f-gripper_articulated, 13 links, 12 joints
Joints:
- joint palm_finger_middle_joint: limit (none) -> lower=-0.16 upper=0.25 effort=100 velocity=100; type fixed -> revolute

File: models/starfish/starfish2.urdf (robot description, URDF)
Before this commit: robot starfish, 1 links, 0 joints
Links:
- link base_link: geometry collision mesh filename=package://starfish/starfish2_vhacd.obj scale=.35 .35 .35; visual mesh filename=package://starfish/starfish2_vhacd.dae scale=.35 .35 .35
