Commit message: starfish demo data recorded - 100 frames

File: models/starfish/starfish2.urdf (robot description, URDF)
Before this commit: robot starfish, 1 links, 0 joints
Links:
- link base_link: geometry collision mesh filename=package://starfish/starfish2_vhacd.obj scale=.5 .5 .5; visual mesh filename=package://starfish/starfish2_vhacd.dae scale=.5 .5 .5

Commit message: added visualization.py; starfish demo

File: models/starfish/starfish2.urdf (robot description, URDF)
Before this commit: robot starfish, 1 links, 0 joints
Links:
- link base_link: geometry collision mesh filename=package://starfish/starfish2_vhacd.obj scale=.4 .4 .4; visual mesh filename=package://starfish/starfish2_vhacd.dae scale=.4 .4 .4
