Commit message: 3-link fish added and data recorded for Blender

File: models/fine-fish/fine-fish.urdf (robot description, URDF)
Before this commit: robot fish, 2 links, 1 joints
Joints:
- joint joint1: limit lower=-1.5 upper=1.5 effort=20 velocity=0.2 -> lower=-1.5 upper=1.5 effort=1000 velocity=0.2
