Commit message: shovel-fish worked in planner and blender

File: models/fine-fish-10/fine-fish-10.urdf (robot description, URDF)
Before this commit: robot fish, 10 links, 9 joints
Links:
- link p1: mass 100 -> 60
- link p10: mass 100 -> 200
- link p2: mass 100 -> 60
- link p3: mass 100 -> 70
- link p4: mass 100 -> 80
- link p5: mass 100 -> 90
- link p7: mass 100 -> 120
- link p8: mass 100 -> 140
- link p9: mass 100 -> 160
