Commit message: starfish urdf updated

File: models/starfish-soft/starfish-soft-16dof.urdf (robot description, URDF)
Before this commit: robot starfish, 11 links, 10 joints
Links:
- link arm1: mass 100 -> 50
- link arm2: mass 100 -> 50
- link arm3: mass 100 -> 50
- link arm4: mass 100 -> 50
- link arm5: mass 100 -> 50
- link mid1: mass 10 -> 1
- link mid2: mass 10 -> 1
- link mid3: mass 10 -> 1
- link mid4: mass 10 -> 1
- link mid5: mass 10 -> 1

Commit message: test04 band-hourglass num_ctrl_points halfdone

File: models/starfish-soft/starfish-soft-16dof.urdf (robot description, URDF)
Before this commit: robot starfish, 11 links, 10 joints
Joints:
- joint joint12: limit lower=-1.5 upper=1.5 effort=1000 velocity=50 -> lower=-.5 upper=.5 effort=1000 velocity=50
